File: hardware/analog_front_end_shield/analog_front_end_shield.kicad_sch (KiCad schematic)
At the start: 48 parts, among them J1 640456-3, J2 S3B-EH(LF)(SN), J3 Conn_01x08, J4 Conn_01x06, J6 Conn_01x10, J7 Conn_01x08, J8 PPTC062LFBN-RC, U1 LMT84LPM, U2 TLV2472AIP

Commit message: AFE board version correction
Parts:
- U1: PN LMT84LPM -> ${VALUE}
Connections:
- net ENC_A: now also J7.4 (Pin_4); no longer J7.5 (Pin_5)
- net ENC_B: now also J7.5 (Pin_5), J8.10 (Pin_10); no longer J7.4 (Pin_4), J8.6 (Pin_6)
- net ENC_SW: now also J8.6 (Pin_6); no longer J8.10 (Pin_10)
- no-connect marks 11 -> 16
Other:
- company: Electronics Student Workshop -> (none)
- title: Analog Front End (AFE) Sheild -> (none)
- moved on the sheet: C6, C7, C8, ENC1, J6, R16, R17, R18, R7, R8, R9

Commit message: Update resistor values for amplifier circuit.
Parts:
- C2: PN K104Z15Y5VF5TL2 -> FG18X7R1E105KRT06
- J3, J7: PN M20-9770846 -> (none)
- R13, R14, R3, R5, R6: value 10K -> 10.2K; PN MFR-25FTF52-10K -> MFR-25FTE52-10K2
- R15: value 6.98K -> 7.15K
Other:
- note added: "V_{OUT(MAX)} = 2.044V V_{OUT(MIN)} = 62mV"
- note removed: "V_{OUT(MAX)} = 2.039V V_{OUT(MIN)} = 61.7mV"
